File: hardware/commpack.kicad_pcb (KiCad board)
At the start: 2 copper layers, 103.8 x 62.5 mm, 31 parts, among them J1 1240COMM, J2 1240COMM_EXT, J3 L8BE-1G1T-91A, U1 SC16C550B, U2 SST39SF010A, U3 HCF4010, U4 AP1117-33, U5 FT230XS, Y1 22.1184M

Commit message: Some WIP on the UART board.
I don't actually know what changed; this was months ago.
Parts:
- removed J2: 1240COMM_EXT, ether1240:ATA_HEADER
- moved A1 27.2 mm to (160.8, 95.6), turned to 90 degrees
- moved Y1 21.8 mm to (180.7, 108.0)
- moved C1 21.8 mm to (180.9, 111.8)
- moved C2 21.8 mm to (185.5, 111.8)
- moved C4 21.7 mm to (187.4, 93.0)
- moved U1 21.7 mm to (185.2, 100.2)
- moved U2 18.0 mm to (202.6, 90.7)
- moved R3 13.8 mm to (150.0, 70.3)
- moved U3 13.8 mm to (164.0, 77.3)
- moved U5 13.8 mm to (133.7, 67.6)
- moved C6 13.8 mm to (144.9, 77.3)
- moved C7 13.8 mm to (139.8, 77.3)
- moved R1 13.8 mm to (139.8, 70.3)
- moved R2 13.8 mm to (144.9, 70.3)
- moved R4 13.8 mm to (155.1, 70.3)
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Connections:
- net Net-(A1-PadB10) renamed /E-TX+
- net Net-(A1-PadB11) renamed /E-RX-
- net Net-(A1-PadB12) renamed /E-RX+
- net Net-(A1-PadB13) renamed /E-LED1
- net Net-(A1-PadB14) renamed /E-LED2
- net Net-(A1-PadB9) renamed /E-TX-
- J1 pad A12: /H-FREQ -> (no net)
Routing:
- net GND: track 411.4 -> 19.1 mm, vias 20 -> 3
- net Earth_Protective: track 510.5 -> 320.8 mm, vias 2 -> 0
- net VCC: track 138.2 -> 7.81 mm, vias 8 -> 0
- net /H-A7: track 101.5 -> 2.79 mm, vias 4 -> 0
- net /H-A5: track 101.3 -> 7.86 mm, vias 3 -> 1
- net /H-A3: track 98.9 -> 8.00 mm, vias 4 -> 0
- net /H-A1: track 108.1 -> 18.7 mm, vias 5 -> 0
- net /H-A9: track 88.3 -> 0.00 mm, vias 2 -> 0
- net /H-A11: track 74.2 -> 0.00 mm, vias 3 -> 0
- net /H-A0: track 92.9 -> 20.7 mm, vias 5 -> 1
- net +3V3: track 69.1 -> 0.00 mm
- net /H-A2: track 92.0 -> 24.7 mm, vias 3 -> 0
- net /H-A6: track 74.3 -> 7.12 mm, vias 3 -> 0
- net /H-A4: track 75.8 -> 10.0 mm, vias 2 -> 0
- net /H-A8: track 65.5 -> 0.00 mm, vias 2 -> 0
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Other:
- board text removed: "+5"
- board text removed: "A0"
- board text removed: "A1"
- board text removed: "A10"
- board text removed: "A11"
- board text removed: "A12"
- board text removed: "A13"
- board text removed: "A2"
- board text removed: "A3"
- board text removed: "A4"
- board text removed: "A5"
- board text removed: "A6"
- board text removed: "A7"
- board text removed: "A8"
- board text removed: "A9"
- board text removed: "D0"
- board text removed: "D1"
- board text removed: "D2"
- board text removed: "D3"
- board text removed: "D4"
- board text removed: "D5"
- board text removed: "D6"
- board text removed: "D7"
- board text removed: "G"
- board text removed: "GND"
- board text removed: "INT"
- board text removed: "OSC"
- board text removed: "PE"
- board text removed: "RST"
- board text removed: "USE ATA RIBBON"
- board text removed: "~CS"
- board text removed: "~RD"
- board text removed: "~RS"
- board text removed: "~WR"

Commit message: Rename local libraries.
Parts:
- A1: footprint ether1240:Omega2 -> local:Omega2
- Bonsai: footprint ether1240:Bonsai -> local:Bonsai
- G***: footprint ether1240:OSHW -> local:OSHW
- H1, H2, H3, H4: footprint ether1240:MountingHole_140mil_Pad -> local:MountingHole_140mil_Pad
- J1: footprint ether1240:1240COMM -> local:1240COMM
- J3: footprint ether1240:L8BE-1G1T-91A -> local:L8BE-1G1T-91A
- U2: footprint ether1240:PLCC-32_THT-Socket -> local:PLCC-32_THT-Socket
Changed lines of the file:
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@@
     (add_net VCC)
   )
-  (module ether1240:MountingHole_140mil_Pad (layer F.Cu)
+  (module local:MountingHole_140mil_Pad (layer F.Cu)
     (at 210.82 113.665)
     (descr "Mounting Hole 140mil")
@@
       (solder_mask_margin 0.5) (clearance 0.5))
   )
-  (module ether1240:MountingHole_140mil_Pad (layer F.Cu)
+  (module local:MountingHole_140mil_Pad (layer F.Cu)
     (at 125.73 113.665)
     (descr "Mounting Hole 140mil")
@@
       (net 2 Earth_Protective))
   )
-  (module ether1240:MountingHole_140mil_Pad (layer F.Cu)
+  (module local:MountingHole_140mil_Pad (layer F.Cu)
     (at 125.73 64.135)
     (descr "Mounting Hole 140mil")
@@
       (net 2 Earth_Protective))
   )
-  (module ether1240:MountingHole_140mil_Pad (layer F.Cu)
+  (module local:MountingHole_140mil_Pad (layer F.Cu)
     (at 210.82 64.135)
     (descr "Mounting Hole 140mil")
@@
       (net 2 Earth_Protective))
   )
-  (module ether1240:Omega2 (layer F.Cu)
+  (module local:Omega2 (layer F.Cu)
     (at 160.79 95.59 90)
     (fp_text reference A1 (at 0 -14.5 90) (layer F.SilkS)
@@
     )
   )
-  (module ether1240:1240COMM locked (layer F.Cu)
+  (module local:1240COMM locked (layer F.Cu)
     (at 214.249 88.9)
     (fp_text reference J1 (at 2.54 0 90) (layer F.SilkS)
@@
       (net 1 GND))
   )
-  (module ether1240:L8BE-1G1T-91A (layer F.Cu)
+  (module local:L8BE-1G1T-91A (layer F.Cu)
     (at 121.92 98.425 270)
     (fp_text reference J3 (at 0.0254 -23.9776 270) (layer F.SilkS)
@@
       (net 55 /E-RX+))
   )
-  (module ether1240:PLCC-32_THT-Socket (layer F.Cu)
+  (module local:PLCC-32_THT-Socket (layer F.Cu)
     (at 202.565 90.678)
     (descr "PLCC, 32 pins, through hole")
@@
     )
   )
-  (module ether1240:OSHW locked (layer B.Cu)
+  (module local:OSHW locked (layer B.Cu)
     (at 170.18 102.87 180)
     (fp_text reference G*** (at 0 -6.73608 180) (layer B.SilkS) hide
@@
       (xy 4.22656 -5.3721) (xy 4.0386 -5.54482) (xy 3.90652 -5.66166) (xy 3.85064 -5.70484)) (layer B.SilkS) (width 0.00254))
   )
-  (module ether1240:Bonsai locked (layer F.Cu)
+  (module local:Bonsai locked (layer F.Cu)
     (at 155.575 104.14)
     (descr "Imported from Bonsai.svg")
