File: hardware/commpack.sch (KiCad schematic (older format))
At the start: 18 parts, among them J1 1240COMM, J2 1240COMM_EXT, J3 L8BE-1G1T-91A, U1 SC16C550B, U2 SST39SF010A, U3 HCF4010, U4 AP1117-33, Y1 22.1184M

Commit message: Switch Y1 to through-hole footprint.
Parts:
- added unit 2 of U3
- added unit 7 of U3
- Y1: footprint Crystals:Crystal_SMD_HC49-SD_HandSoldering -> Crystals:Crystal_HC49-U_Vertical
Connections:
- net +3V3: now also U3.1 (VCC)
- net A-RX: now also A1.A8 (GPIO46/UART1_RX), U3.4; no longer U1.8 (TX)
- net A-~CTS: now also A1.A7 (GPIO15), U3.2; no longer U1.32 (~RTS)
- net GND: now also U3.8 (GND)
- net VCC: now also U3.16 (VDD)
- net U-~RTS: now reaches U3.3
- net U-~RTS: now also U1.32 (~RTS)
- new net U-TX: U1.8 (TX), U3.5
- no-connect marks 34 -> 26
Other:
- moved on the sheet: U3A
Changed lines of the file:
@@
 F 0 "Y1" H 1700 3750 50  0000 C CNN
 F 1 "22.1184M" H 1700 3450 50  0000 C CNN
-F 2 "Crystals:Crystal_SMD_HC49-SD_HandSoldering" H 1700 3600 50  0001 C CNN
+F 2 "Crystals:Crystal_HC49-U_Vertical" H 1700 3600 50  0001 C CNN
 F 3 "" H 1700 3600 50  0001 C CNN
 	1    1700 3600
@@
 	3200 1300 2850 1300
 Text Label 2650 800  2    60   ~ 0
-A-RX
+U-TX
 Wire Wire Line
 	1100 2600 550  2600
@@
 	2300 2600 2650 2600
 Text Label 2650 2600 2    60   ~ 0
-A-~CTS
+U-~RTS
 Text Label 550  2600 0    60   ~ 0
 A-~RTS
@@
 Flash ROM
 Wire Wire Line
-	6250 1550 6750 1550
-Wire Wire Line
-	6250 1450 6750 1450
-Wire Wire Line
 	6750 1350 6350 1350
 Text Label 6350 1350 0    60   ~ 0
 A-~RTS
-Text Label 5100 1450 0    60   ~ 0
+Text Label 6350 1450 0    60   ~ 0
 A-~CTS
-Text Label 5100 1550 0    60   ~ 0
+Text Label 6350 1550 0    60   ~ 0
 A-RX
 $Comp
@@
 Text Label 550  800  0    60   ~ 0
 A-TX
-Wire Wire Line
-	6750 1650 6350 1650
-Text Label 6350 1650 0    60   ~ 0
-A-TX
 $Comp
 L C C4
@@
 L HCF4010 U3
 U 1 1 5A72DF90
-P 5850 1850
-F 0 "U3" H 5850 1520 60  0000 C CNN
-F 1 "HCF4010" H 5850 1600 60  0000 C CNN
-F 2 "Housings_SOIC:SOIC-16_3.9x9.9mm_Pitch1.27mm" H 5850 1900 60  0001 C CNN
-F 3 "" H 5850 1900 60  0001 C CNN
-	1    5850 1850
-	1    0    0    -1
-$EndComp
-Wire Wire Line
-	5450 1450 5100 1450
-Wire Wire Line
-	5450 1550 5100 1550
+P 6000 1350
+F 0 "U3" H 6000 1250 60  0000 C CNN
+F 1 "HCF4010" H 6000 1170 60  0001 C CNN
+F 2 "Housings_SOIC:SOIC-16_3.9x9.9mm_Pitch1.27mm" H 6000 1500 60  0001 C CNN
+F 3 "" H 6000 1500 60  0001 C CNN
+	1    6000 1350
+	1    0    0    -1
+$EndComp
 $Comp
 L +3V3 #PWR023
 U 1 1 5A72EA03
-P 5950 950
-F 0 "#PWR023" H 5950 800 50  0001 C CNN
-F 1 "+3V3" H 5950 1090 50  0000 C CNN
-F 2 "" H 5950 950 50  0001 C CNN
-F 3 "" H 5950 950 50  0001 C CNN
-	1    5950 950
+P 5850 2450
+F 0 "#PWR023" H 5850 2300 50  0001 C CNN
+F 1 "+3V3" H 5850 2590 50  0000 C CNN
+F 2 "" H 5850 2450 50  0001 C CNN
+F 3 "" H 5850 2450 50  0001 C CNN
+	1    5850 2450
 	1    0    0    -1
 $EndComp
@@
 L VCC #PWR024
 U 1 1 5A72EA3B
-P 5750 950
-F 0 "#PWR024" H 5750 800 50  0001 C CNN
-F 1 "VCC" H 5750 1100 50  0000 C CNN
-F 2 "" H 5750 950 50  0001 C CNN
-F 3 "" H 5750 950 50  0001 C CNN
-	1    5750 950
-	1    0    0    -1
-$EndComp
-NoConn ~ 5450 1650
-NoConn ~ 5450 1750
-NoConn ~ 5450 1850
-NoConn ~ 5450 1950
-NoConn ~ 6250 1950
-NoConn ~ 6250 1850
-NoConn ~ 6250 1750
-NoConn ~ 6250 1650
+P 5650 2450
+F 0 "#PWR024" H 5650 2300 50  0001 C CNN
+F 1 "VCC" H 5650 2600 50  0000 C CNN
+F 2 "" H 5650 2450 50  0001 C CNN
+F 3 "" H 5650 2450 50  0001 C CNN
+	1    5650 2450
+	1    0    0    -1
+$EndComp
+Text Label 6350 1650 0    60   ~ 0
+A-TX
+Wire Wire Line
+	6750 1650 6350 1650
+$Comp
+L HCF4010 U3
+U 2 1 5A73EC5D
+P 6000 1650
+F 0 "U3" H 6000 1550 60  0000 C CNN
+F 1 "HCF4010" H 6000 1470 60  0001 C CNN
+F 2 "Housings_SOIC:SOIC-16_3.9x9.9mm_Pitch1.27mm" H 6000 1800 60  0001 C CNN
+F 3 "" H 6000 1800 60  0001 C CNN
+	2    6000 1650
+	1    0    0    -1
+$EndComp
+$Comp
+L HCF4010 U3
+U 7 1 5A73F4F4
+P 5750 2850
+F 0 "U3" H 5750 2750 60  0000 C CNN
+F 1 "HCF4010" H 5750 2670 60  0001 C CNN
+F 2 "Housings_SOIC:SOIC-16_3.9x9.9mm_Pitch1.27mm" H 5750 3000 60  0001 C CNN
+F 3 "" H 5750 3000 60  0001 C CNN
+	7    5750 2850
+	1    0    0    -1
+$EndComp
+Wire Wire Line
+	6250 1450 6750 1450
+Wire Wire Line
+	6250 1550 6750 1550
+Wire Wire Line
+	6250 1450 6250 1350
+Wire Wire Line
+	6250 1350 6200 1350
+Wire Wire Line
+	6250 1550 6250 1650
+Wire Wire Line
+	6250 1650 6200 1650
+Wire Wire Line
+	5800 1350 5450 1350
+Wire Wire Line
+	5800 1650 5450 1650
+Text Label 5450 1350 0    60   ~ 0
+U-~RTS
+Text Label 5450 1650 0    60   ~ 0
+U-TX
 $EndSCHEMATC

Commit message: Update schematic to KiCAD 5.0.
Parts:
- added C6, C7: 47p, Capacitors_SMD:C_0805_HandSoldering, symbol Device:C
- added J4: USB_B, symbol Connector:USB_B
- added R1, R2: 27R, Resistors_SMD:R_2010_HandSoldering, symbol Device:R
- added R3: 4k7, Resistors_SMD:R_2010_HandSoldering, symbol Device:R
- added R4: 10k, Resistors_SMD:R_2010_HandSoldering, symbol Device:R
- added U5: FT230XS, Housings_SSOP:SSOP-16_3.9x4.9mm_Pitch0.635mm, symbol ether1240:FT230XS
- A1: symbol Omega2+ -> ether1240:Omega2+
- C1, C2, C3, C4, C5: symbol C -> Device:C
- H1, H2, H3, H4: symbol Screw_Terminal_01x01 -> Connector:Screw_Terminal_01x01
- J1: symbol 1240COMM -> ether1240:1240COMM
- J2: symbol 1240COMM_EXT -> ether1240:1240COMM_EXT
- J3: symbol L8BE-1G1T-91A -> ether1240:L8BE-1G1T-91A
- U1: symbol SC16C550B -> ether1240:SC16C550B
- U2: symbol SST39SF010A -> ether1240:SST39SF010A
- U3: symbol HCF4010 -> ether1240:HCF4010
- U4: symbol AP1117-33 -> Regulator_Linear:AP1117-33
- Y1: symbol Crystal -> Device:Crystal
Connections:
- net labels added: E-LED1, E-LED2, E-RX+, E-RX-, E-TX+, E-TX-
- wire segments 170 -> 234
- no-connect marks 26 -> 29
Other:
- note added: "Ethernet"
- note added: "USB UART"
- moved on the sheet: A1, H1, H2, H3, H4, J3, U3A, U3B, U3G

Commit message: Some WIP on the UART board.
I don't actually know what changed; this was months ago.
Parts:
- removed J2: 1240COMM_EXT, ether1240:ATA_HEADER, symbol ether1240:1240COMM_EXT
Connections:
- net labels removed: H-FREQ
- wire segments 234 -> 201
- no-connect marks 29 -> 30
Other:
- note added: "Host Bus Connector"
- note removed: "Host Bus Connectors"
Changed lines of the file:
@@
 Text Label 2200 7000 0    60   ~ 0
 H-A13
-Entry Wire Line
-	2750 5700 2650 5800
-Entry Wire Line
-	2750 5800 2650 5900
-Entry Wire Line
-	2750 5900 2650 6000
-Entry Wire Line
-	2750 6000 2650 6100
-Entry Wire Line
-	2750 6100 2650 6200
-Entry Wire Line
-	2750 6200 2650 6300
-Entry Wire Line
-	2750 6300 2650 6400
-Entry Wire Line
-	2750 6400 2650 6500
-Entry Wire Line
-	2750 6500 2650 6600
-Entry Wire Line
-	2750 6600 2650 6700
-Entry Wire Line
-	2750 6700 2650 6800
-Entry Wire Line
-	2750 6800 2650 6900
-Entry Wire Line
-	2750 6900 2650 7000
-Entry Wire Line
-	2750 7000 2650 7100
-Text Label 3100 5700 2    60   ~ 0
-H-A0
-Text Label 3100 5800 2    60   ~ 0
-H-A1
-Text Label 3100 5900 2    60   ~ 0
-H-A2
-Text Label 3100 6000 2    60   ~ 0
-H-A3
-Text Label 3100 6100 2    60   ~ 0
-H-A4
-Text Label 3100 6200 2    60   ~ 0
-H-A5
-Text Label 3100 6300 2    60   ~ 0
-H-A6
-Text Label 3100 6400 2    60   ~ 0
-H-A7
-Text Label 3100 6500 2    60   ~ 0
-H-A8
-Text Label 3100 6600 2    60   ~ 0
-H-A9
-Text Label 3100 6700 2    60   ~ 0
-H-A10
-Text Label 3100 6800 2    60   ~ 0
-H-A11
-Text Label 3100 6900 2    60   ~ 0
-H-A12
-Text Label 3100 7000 2    60   ~ 0
-H-A13
-Entry Wire Line
-	4750 5300 4650 5400
-Entry Wire Line
-	4750 5400 4650 5500
-Entry Wire Line
-	4750 5500 4650 5600
-Entry Wire Line
-	4750 5600 4650 5700
-Entry Wire Line
-	4750 5700 4650 5800
-Entry Wire Line
-	4750 5800 4650 5900
-Entry Wire Line
-	4750 5900 4650 6000
-Entry Wire Line
-	4750 6000 4650 6100
-Text Label 4550 5400 2    60   ~ 0
-H-D0
-Text Label 4550 5500 2    60   ~ 0
-H-D1
-Text Label 4550 5600 2    60   ~ 0
-H-D2
-Text Label 4550 5700 2    60   ~ 0
-H-D3
-Text Label 4550 5800 2    60   ~ 0
-H-D4
-Text Label 4550 5900 2    60   ~ 0
-H-D5
-Text Label 4550 6000 2    60   ~ 0
-H-D6
-Text Label 4550 6100 2    60   ~ 0
-H-D7
-$Comp
-L power:GND #PWR11
-U 1 1 59FE6FF1
-P 3850 7400
-F 0 "#PWR11" H 3850 7150 50  0001 C CNN
-F 1 "GND" H 3850 7250 50  0000 C CNN
-F 2 "" H 3850 7400 50  0001 C CNN
-F 3 "" H 3850 7400 50  0001 C CNN
-	1    3850 7400
-	-1   0    0    -1
-$EndComp
-$Comp
-L power:Earth_Protective #PWR12
-U 1 1 59FE6FF7
-P 4100 7400
-F 0 "#PWR12" H 4350 7150 50  0001 C CNN
-F 1 "Earth_Protective" H 4550 7250 50  0001 C CNN
-F 2 "" H 4100 7300 50  0001 C CNN
-F 3 "" H 4100 7300 50  0001 C CNN
-	1    4100 7400
-	-1   0    0    -1
-$EndComp
 $Comp
 L Connector:Screw_Terminal_01x01 H1
@@
 $EndComp
 Text Notes 550  4400 0    60   ~ 0
-Host Bus Connectors
+Host Bus Connector
 $Comp
 L Regulator_Linear:AP1117-33 U4
@@
 NoConn ~ 8050 4100
 NoConn ~ 8050 4200
-$Comp
-L ether1240:1240COMM_EXT J2
-U 1 1 5A02D637
-P 3650 6000
-F 0 "J2" V 3750 6000 60  0000 C CNN
-F 1 "1240COMM_EXT" V 3650 6000 60  0000 C CNN
-F 2 "ether1240:ATA_HEADER" H 4050 7650 60  0001 C CNN
-F 3 "" H 4050 7650 60  0001 C CNN
-	1    3650 6000
-	1    0    0    -1
-$EndComp
 NoConn ~ 1450 4800
 $Comp
@@
 $EndComp
 $Comp
-L power:VCC #PWR10
-U 1 1 5A2F4D96
-P 3850 4800
-F 0 "#PWR10" H 3850 4650 50  0001 C CNN
-F 1 "VCC" H 3850 4950 50  0000 C CNN
-F 2 "" H 3850 4800 50  0001 C CNN
-F 3 "" H 3850 4800 50  0001 C CNN
-	1    3850 4800
-	1    0    0    -1
-$EndComp
-$Comp
 L power:VCC #PWR15
 U 1 1 5A2F4DC6
@@
 	1    0    0    -1
 $EndComp
-Text Label 2200 4550 0    60   ~ 0
-H-FREQ
 NoConn ~ 6350 4000
 NoConn ~ 6350 4100
@@
 Connection ~ 1250 3600
 Wire Wire Line
-	3950 4550 3950 4800
-Wire Wire Line
-	1350 4550 3950 4550
-Wire Wire Line
-	1350 4800 1350 4550
-Wire Wire Line
 	6150 7000 6300 7000
 Wire Wire Line
@@
 Wire Wire Line
 	8050 4000 8050 3800
-Wire Wire Line
-	3150 5500 2150 5500
-Wire Wire Line
-	2150 5400 3150 5400
-Wire Wire Line
-	2150 5300 3150 5300
-Wire Wire Line
-	2150 5200 3150 5200
-Wire Wire Line
-	2150 5100 3150 5100
 Connection ~ 6300 7000
 Wire Wire Line
@@
 	1200 7350 1200 7400
 Wire Wire Line
-	3150 5700 2750 5700
-Wire Wire Line
-	3150 5800 2750 5800
-Wire Wire Line
-	3150 5900 2750 5900
-Wire Wire Line
-	3150 6000 2750 6000
-Wire Wire Line
-	3150 6100 2750 6100
-Wire Wire Line
-	3150 6200 2750 6200
-Wire Wire Line
-	3150 6300 2750 6300
-Wire Wire Line
-	3150 6400 2750 6400
-Wire Wire Line
-	3150 6500 2750 6500
-Wire Wire Line
-	3150 6600 2750 6600
-Wire Wire Line
-	3150 6700 2750 6700
-Wire Wire Line
-	3150 6800 2750 6800
-Wire Wire Line
-	3150 6900 2750 6900
-Wire Wire Line
-	3150 7000 2750 7000
-Wire Wire Line
-	4250 5400 4650 5400
-Wire Wire Line
-	4250 5500 4650 5500
-Wire Wire Line
-	4250 5600 4650 5600
-Wire Wire Line
-	4250 5700 4650 5700
-Wire Wire Line
-	4250 5800 4650 5800
-Wire Wire Line
-	4250 5900 4650 5900
-Wire Wire Line
-	4250 6000 4650 6000
-Wire Wire Line
-	4250 6100 4650 6100
-Wire Wire Line
-	3850 7300 3850 7400
-Wire Wire Line
-	3950 7300 3950 7350
-Wire Wire Line
-	3950 7350 4100 7350
-Wire Wire Line
-	4100 7350 4100 7400
-Wire Wire Line
-	650  6300 650  7700
-Wire Wire Line
-	4300 7700 4300 6300
-Wire Wire Line
-	4300 6300 4250 6300
-Wire Wire Line
 	650  6300 1050 6300
-Wire Wire Line
-	650  7700 4300 7700
 Wire Notes Line
 	4900 4250 500  4250
@@
 Wire Wire Line
 	9250 950  9250 1250
+Entry Wire Line
+	550  6200 650  6300
+Wire Wire Line
+	2150 5100 2550 5100
+Wire Wire Line
+	2150 5200 2550 5200
+Wire Wire Line
+	2150 5300 2550 5300
+Wire Wire Line
+	2150 5400 2550 5400
+Wire Wire Line
+	2150 5500 2550 5500
+Entry Wire Line
+	2550 5100 2650 5200
+Entry Wire Line
+	2550 5200 2650 5300
+Entry Wire Line
+	2550 5300 2650 5400
+Entry Wire Line
+	2550 5400 2650 5500
+Entry Wire Line
+	2550 5500 2650 5600
+NoConn ~ 1350 4800
 Wire Bus Line
-	550  5050 550  6000
+	550  5050 550  6200
 Wire Bus Line
-	4750 5050 4750 6000
-Wire Bus Line
-	2650 5800 2650 7350
+	2650 5200 2650 7350
 $EndSCHEMATC

Commit message: Rename local libraries.
Parts:
- A1: footprint ether1240:Omega2 -> local:Omega2; symbol ether1240:Omega2+ -> local:Omega2+
- H1, H2, H3, H4: footprint ether1240:MountingHole_140mil_Pad -> local:MountingHole_140mil_Pad
- J1: footprint ether1240:1240COMM -> local:1240COMM; symbol ether1240:1240COMM -> local:1240COMM
- J3: footprint ether1240:L8BE-1G1T-91A -> local:L8BE-1G1T-91A; symbol ether1240:L8BE-1G1T-91A -> local:L8BE-1G1T-91A
- U1: symbol ether1240:SC16C550B -> local:SC16C550B
- U2: footprint ether1240:PLCC-32_THT-Socket -> local:PLCC-32_THT-Socket; symbol ether1240:SST39SF010A -> local:SST39SF010A
- U3: symbol ether1240:HCF4010 -> local:HCF4010
- U5: symbol ether1240:FT230XS -> local:FT230XS
Changed lines of the file:
@@
 F 0 "H1" H 9550 1050 50  0000 C CNN
 F 1 "Mount" H 9550 850 50  0000 C CNN
-F 2 "ether1240:MountingHole_140mil_Pad" H 9550 950 50  0001 C CNN
+F 2 "local:MountingHole_140mil_Pad" H 9550 950 50  0001 C CNN
 F 3 "" H 9550 950 50  0001 C CNN
 	1    9550 950
@@
 F 0 "H2" H 9550 1350 50  0000 C CNN
 F 1 "Mount" H 9550 1150 50  0000 C CNN
-F 2 "ether1240:MountingHole_140mil_Pad" H 9550 1250 50  0001 C CNN
+F 2 "local:MountingHole_140mil_Pad" H 9550 1250 50  0001 C CNN
 F 3 "" H 9550 1250 50  0001 C CNN
 	1    9550 1250
@@
 F 0 "H3" H 10100 1050 50  0000 C CNN
 F 1 "Mount" H 10100 850 50  0000 C CNN
-F 2 "ether1240:MountingHole_140mil_Pad" H 10100 950 50  0001 C CNN
+F 2 "local:MountingHole_140mil_Pad" H 10100 950 50  0001 C CNN
 F 3 "" H 10100 950 50  0001 C CNN
 	1    10100 950
@@
 F 0 "H4" H 10100 1350 50  0000 C CNN
 F 1 "Mount" H 10100 1150 50  0000 C CNN
-F 2 "ether1240:MountingHole_140mil_Pad" H 10100 1250 50  0001 C CNN
+F 2 "local:MountingHole_140mil_Pad" H 10100 1250 50  0001 C CNN
 F 3 "" H 10100 1250 50  0001 C CNN
 	1    10100 1250
@@
 Power
 $Comp
-L ether1240:L8BE-1G1T-91A J3
+L local:L8BE-1G1T-91A J3
 U 1 1 5A14541E
 P 10750 5500
 F 0 "J3" H 10850 6100 50  0000 L CNN
 F 1 "L8BE-1G1T-91A" H 10700 6100 50  0000 R CNN
-F 2 "ether1240:L8BE-1G1T-91A" H 10750 5500 50  0001 C CNN
+F 2 "local:L8BE-1G1T-91A" H 10750 5500 50  0001 C CNN
 F 3 "" H 10750 5500 50  0001 C CNN
 	1    10750 5500
@@
 $EndComp
 $Comp
-L ether1240:Omega2+ A1
+L local:Omega2+ A1
 U 1 1 5A1FF68F
 P 7200 4650
 F 0 "A1" H 7200 5500 60  0000 C CNN
 F 1 "Omega2+" H 7200 3800 60  0000 C CNN
-F 2 "ether1240:Omega2" H 7200 4850 60  0001 C CNN
+F 2 "local:Omega2" H 7200 4850 60  0001 C CNN
 F 3 "" H 7200 4850 60  0001 C CNN
 	1    7200 4650
@@
 NoConn ~ 1450 4800
 $Comp
-L ether1240:1240COMM J1
+L local:1240COMM J1
 U 1 1 59FE52B4
 P 1650 6000
 F 0 "J1" V 1550 6000 60  0000 C CNN
 F 1 "1240COMM" V 1650 6000 60  0000 C CNN
-F 2 "ether1240:1240COMM" H 2050 7650 60  0001 C CNN
+F 2 "local:1240COMM" H 2050 7650 60  0001 C CNN
 F 3 "" H 2050 7650 60  0001 C CNN
 	1    1650 6000
@@
 H-RST
 $Comp
-L ether1240:SC16C550B U1
+L local:SC16C550B U1
 U 1 1 5A2ED667
 P 1700 2000
@@
 $EndComp
 $Comp
-L ether1240:SST39SF010A U2
+L local:SST39SF010A U2
 U 1 1 5A2F0DF1
 P 3800 2300
 F 0 "U2" H 3800 3450 60  0000 C CNN
 F 1 "SST39SF010A" H 3825 1150 60  0000 C CNN
-F 2 "ether1240:PLCC-32_THT-Socket" H 3800 2300 60  0001 C CNN
+F 2 "local:PLCC-32_THT-Socket" H 3800 2300 60  0001 C CNN
 F 3 "" H 3800 2300 60  0001 C CNN
 	1    3800 2300
@@
 $EndComp
 $Comp
-L ether1240:HCF4010 U3
+L local:HCF4010 U3
 U 1 1 5A72DF90
 P 5600 4400
@@
 A-TX
 $Comp
-L ether1240:HCF4010 U3
+L local:HCF4010 U3
 U 2 1 5A73EC5D
 P 5600 4700
@@
 $EndComp
 $Comp
-L ether1240:HCF4010 U3
+L local:HCF4010 U3
 U 7 1 5A73F4F4
 P 10800 1300
@@
 U-TX
 $Comp
-L ether1240:FT230XS U5
+L local:FT230XS U5
 U 1 1 5A8E0603
 P 9700 4200
